File: DraaiBoard/DraaiBoard.sch (KiCad schematic (older format))
At the start: 79 parts, among them IC1 ATMEGA8A-P, J1 DB25, K1 RELAY_2RT, K2 RELAY_2RT, K3 RELAY_2RT, K4 RELAY_2RT, K5 RELAY_2RT, K6 RELAY_2RT, K7 RELAY_2RT, K8 RELAY_2RT, K9 RELAY_2RT, P1 CONN_5X2, Q1 BD680, Q10 BC546, Q11 BC546, Q12 BC546, Q13 BC546, Q14 BC546, Q15 BC546, Q2 BD679, Q3 BC546, Q4 BC556, Q5 BC546, Q6 BC556, Q7 BC546, Q8 BC546, Q9 BC546, U1 7805, U2 74LS138, U3 POLOLU_A4988, U4 74LS240, U5 C96ABC, X1 Crystal 14.7456MHz

Commit message: Homing aangepast zodat die iets terug draaid als die op het reedcontact staat. + Middendetect aan en uit seperaat
Parts:
- R4: value 220E -> 132E
Changed lines of the file:
@@
 Sheet 1 1
 Title "DraaiPlatform aansturing"
-Date "3 jan 2016"
+Date "3 apr 2016"
 Rev "1.0"
 Comp "Eric"
@@
 P 3750 6400
 F 0 "R4" V 3830 6400 40  0000 C CNN
-F 1 "220E" V 3757 6401 40  0000 C CNN
+F 1 "132E" V 3757 6401 40  0000 C CNN
 F 2 "~" V 3680 6400 30  0000 C CNN
 F 3 "~" H 3750 6400 30  0000 C CNN
